Commit message: rb10_1300e urdf correction

File: rbpodo_description/meshes/rb5_850e/collision/rb5_850e.urdf (robot description, URDF)
Before this commit: robot rb3_1200e, 8 links, 7 joints
Links:
- link link0: geometry collision mesh filename=package://rbpodo_description/meshes/rb5_850e/collision/link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; visual mesh filename=package://rbpodo_description/meshes/rb5_850e/visual/link0.d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
- link link1: mass 4.08789303 -> 4.147; geometry collision mesh filename=package://rbpodo_description/meshes/rb5_850e/collision/link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; visual mesh filename=package://rbpodo_description/meshes/rb5_850e/visual/link1.d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
- link link2: mass 9.63917443 -> 9.633; geometry collision mesh filename=package://rbpodo_description/meshes/rb5_850e/collision/link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; visual mesh filename=package://rbpodo_description/meshes/rb5_850e/visual/link2.d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
- link link3: mass 3.99792153 -> 3.915; geometry collision mesh filename=package://rbpodo_description/meshes/rb5_850e/collision/link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; visual mesh filename=package://rbpodo_description/meshes/rb5_850e/visual/link3.d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
- link link4: mass 1.50851652 -> 1.452; geometry collision mesh filename=package://rbpodo_description/meshes/rb5_850e/collision/link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; visual mesh filename=package://rbpodo_description/meshes/rb5_850e/visual/link4.d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
- link link5: mass 1.50851652 -> 1.454; geometry collision mesh filename=package://rbpodo_description/meshes/rb5_850e/collision/link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; visual mesh filename=package://rbpodo_description/meshes/rb5_850e/visual/link5.d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
- link link6: mass 0.21200156 -> 0.243; geometry collision mesh filename=package://rbpodo_description/meshes/rb5_850e/collision/link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; visual mesh filename=package://rbpodo_description/meshes/rb5_850e/visual/link6.d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
Joints:
- joint elbow: origin xyz=0 -0.1484 0.5669 rpy=0 0 0 -> xyz=0 0 0.425 rpy=0 0 0
- joint wrist1: origin xyz=0 0.1484 0.5224 rpy=0 0 0 -> xyz=0 0 0.392 rpy=0 0 0
- joint wrist2: origin xyz=0 -0.1107 0 rpy=0 0 0 -> xyz=0 -0.1107 0.1107 rpy=0 0 0
- joint wrist3: origin xyz=0 0 0.1107 rpy=0 0 0 -> xyz=0 0 0 rpy=0 0 0

File: rbpodo_description/robots/rb10_1300e.urdf (robot description, URDF)
Before this commit: robot rb10_1300e, 8 links, 7 joints
Joints:
- joint base: origin xyz=0 0 0.197 rpy=0 0 0 -> xyz=0 0 0 rpy=0 0 0
- joint elbow: origin xyz=0 0 0.6127 rpy=0 0 0 -> xyz=0 -0.1875 0.6127 rpy=0 0 0
- joint shoulder: origin xyz=0 -0.1875 0 rpy=0 0 0 -> xyz=0 0 0.197 rpy=0 0 0
- joint wrist1: origin xyz=0 0.11715 0.57015 rpy=0 0 0 -> xyz=0 0.1484 0.57015 rpy=0 0 0
