Commit message: fix: some robot models were added

File: rbpodo_description/robots/rb10_1300e_u.urdf (robot description, URDF)
Before this commit: robot rb20_1900es, 8 links, 7 joints
Links:
- link link0: geometry collision mesh filename=package://rbpodo_description/meshes/rb10_1300e_u/collision/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; visual mesh filename=package://rbpodo_description/meshes/rb10_1300e_u/visual/lin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
- link link1: mass 15.48 -> 8.366; geometry collision mesh filename=package://rbpodo_description/meshes/rb10_1300e_u/collision/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; visual mesh filename=package://rbpodo_description/meshes/rb10_1300e_u/visual/lin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
- link link2: mass 32.79 -> 15.61; geometry collision mesh filename=package://rbpodo_description/meshes/rb10_1300e_u/collision/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; visual mesh filename=package://rbpodo_description/meshes/rb10_1300e_u/visual/lin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
- link link3: mass 8.371 -> 5.69; geometry collision mesh filename=package://rbpodo_description/meshes/rb10_1300e_u/collision/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; visual mesh filename=package://rbpodo_description/meshes/rb10_1300e_u/visual/lin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
- link link4: mass 8.14 -> 2.062; geometry collision mesh filename=package://rbpodo_description/meshes/rb10_1300e_u/collision/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; visual mesh filename=package://rbpodo_description/meshes/rb10_1300e_u/visual/lin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
- link link5: mass 1.924 -> 2.061; geometry collision mesh filename=package://rbpodo_description/meshes/rb10_1300e_u/collision/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; visual mesh filename=package://rbpodo_description/meshes/rb10_1300e_u/visual/lin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
- link link6: mass 0.588 -> 0.406; geometry collision mesh filename=package://rbpodo_description/meshes/rb10_1300e_u/collision/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; visual mesh filename=package://rbpodo_description/meshes/rb10_1300e_u/visual/lin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
Joints:
- joint base: origin xyz=0 0 0.241 rpy=0 0 0 -> xyz=0 0 0 rpy=0 0 0
- joint elbow: origin xyz=0 0 0.885 rpy=0 0 0 -> xyz=0 -0.1875 0.6127 rpy=0 0 0
- joint shoulder: origin xyz=0 -0.2545 0 rpy=0 0 0 -> xyz=0 0 0.197 rpy=0 0 0
- joint tcp_joint: origin xyz=0 0 0.13 rpy=0 0 0 -> xyz=0 -0.1153 0 rpy=0 0 0
- joint wrist1: axis 0 0 1 -> 0 1 0; origin xyz=0 0.1875 0 rpy=0 0 0 -> xyz=0 0.1514 0.57015 rpy=0 0 0
- joint wrist2: axis 0 1 0 -> 0 0 1; origin xyz=0 -0.1292 0.885 rpy=0 0 0 -> xyz=0 -0.11715 0 rpy=0 0 0
- joint wrist3: axis 0 0 1 -> 0 1 0; origin xyz=0 0.1292 0 rpy=0 0 0 -> xyz=0 0 0.11715 rpy=0 0 0

File: rbpodo_description/robots/rb10_1300e_u.urdf.xacro (robot description, xacro)
@@ -1,4 +1,4 @@
 <?xml version='1.0' encoding='utf-8'?>
-<robot xmlns:xacro="http://www.ros.org/wiki/xacro" name="rb20_1900es">
+<robot xmlns:xacro="http://www.ros.org/wiki/xacro" name="rb10_1300e_u">
   <xacro:include filename="$(find rbpodo_description)/robots/rb_6dof.xacro" />
   <xacro:include filename="$(find rbpodo_description)/robots/rb_6dof.ros2_control.xacro" />
@@ -15,5 +15,5 @@
   <xacro:property name="wrist2_tc" value="${1}" />
   <xacro:property name="wrist3_tc" value="${1}" />
-  <xacro:rb_6dof model_id="rb20_1900es" prefix="$(arg prefix)" tcp_name="tcp" tcp_xyz="0 0 0.13" tcp_rpy="0 0 0" />
+  <xacro:rb_6dof model_id="rb10_1300e_u" prefix="$(arg prefix)" tcp_name="tcp" tcp_xyz="0 -0.1153 0" tcp_rpy="0 0 0" />
   <xacro:rb_6dof_ros2_control prefix="$(arg prefix)" robot_ip="$(arg robot_ip)" cb_simulation="$(arg cb_simulation)" use_fake_hardware="$(arg use_fake_hardware)" fake_sensor_commands="$(arg fake_sensor_commands)" torque_constants="${[base_tc, shoulder_tc, elbow_tc, wrist1_tc, wrist2_tc, wrist3_tc]}" />
 </robot>

File: rbpodo_description/robots/rb16_900e_u.urdf (robot description, URDF)
Before this commit: robot rb20_1900es, 8 links, 7 joints
Links:
- link link0: geometry collision mesh filename=package://rbpodo_description/meshes/rb16_900e_u/collision/l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; visual mesh filename=package://rbpodo_description/meshes/rb16_900e_u/visual/link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
- link link1: mass 15.48 -> 8.36480574; geometry collision mesh filename=package://rbpodo_description/meshes/rb16_900e_u/collision/l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; visual mesh filename=package://rbpodo_description/meshes/rb16_900e_u/visual/link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
- link link2: mass 32.79 -> 14.65108225; geometry collision mesh filename=package://rbpodo_description/meshes/rb16_900e_u/collision/l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; visual mesh filename=package://rbpodo_description/meshes/rb16_900e_u/visual/link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
- link link3: mass 8.371 -> 4.99600074; geometry collision mesh filename=package://rbpodo_description/meshes/rb16_900e_u/collision/l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; visual mesh filename=package://rbpodo_description/meshes/rb16_900e_u/visual/link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
- link link4: mass 8.14 -> 2.04897826; geometry collision mesh filename=package://rbpodo_description/meshes/rb16_900e_u/collision/l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; visual mesh filename=package://rbpodo_description/meshes/rb16_900e_u/visual/link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
- link link5: mass 1.924 -> 2.05100562; geometry collision mesh filename=package://rbpodo_description/meshes/rb16_900e_u/collision/l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; visual mesh filename=package://rbpodo_description/meshes/rb16_900e_u/visual/link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
- link link6: mass 0.588 -> 0.40590103; geometry collision mesh filename=package://rbpodo_description/meshes/rb16_900e_u/collision/l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; visual mesh filename=package://rbpodo_description/meshes/rb16_900e_u/visual/link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
Joints:
- joint base: origin xyz=0 0 0.241 rpy=0 0 0 -> xyz=0 0 0.197 rpy=0 0 0
- joint elbow: origin xyz=0 0 0.885 rpy=0 0 0 -> xyz=0 0 0.4127 rpy=0 0 0
- joint shoulder: origin xyz=0 -0.2545 0 rpy=0 0 0 -> xyz=0 -0.1875 0 rpy=0 0 0
- joint tcp_joint: origin xyz=0 0 0.13 rpy=0 0 0 -> xyz=0 -0.1153 0 rpy=0 0 0
- joint wrist1: axis 0 0 1 -> 0 1 0; origin xyz=0 0.1875 0 rpy=0 0 0 -> xyz=0 0.1514 0.37015 rpy=0 0 0
- joint wrist2: axis 0 1 0 -> 0 0 1; origin xyz=0 -0.1292 0.885 rpy=0 0 0 -> xyz=0 -0.11715 0 rpy=0 0 0
- joint wrist3: axis 0 0 1 -> 0 1 0; origin xyz=0 0.1292 0 rpy=0 0 0 -> xyz=0 0 0.11715 rpy=0 0 0

File: rbpodo_description/robots/rb16_900e_u.urdf.xacro (robot description, xacro)
@@ -1,4 +1,4 @@
 <?xml version='1.0' encoding='utf-8'?>
-<robot xmlns:xacro="http://www.ros.org/wiki/xacro" name="rb20_1900es">
+<robot xmlns:xacro="http://www.ros.org/wiki/xacro" name="rb16_900e_u">
   <xacro:include filename="$(find rbpodo_description)/robots/rb_6dof.xacro" />
   <xacro:include filename="$(find rbpodo_description)/robots/rb_6dof.ros2_control.xacro" />
@@ -15,5 +15,5 @@
   <xacro:property name="wrist2_tc" value="${1}" />
   <xacro:property name="wrist3_tc" value="${1}" />
-  <xacro:rb_6dof model_id="rb20_1900es" prefix="$(arg prefix)" tcp_name="tcp" tcp_xyz="0 0 0.13" tcp_rpy="0 0 0" />
+  <xacro:rb_6dof model_id="rb16_900e_u" prefix="$(arg prefix)" tcp_name="tcp" tcp_xyz="0 -0.1153 0" tcp_rpy="0 0 0" />
   <xacro:rb_6dof_ros2_control prefix="$(arg prefix)" robot_ip="$(arg robot_ip)" cb_simulation="$(arg cb_simulation)" use_fake_hardware="$(arg use_fake_hardware)" fake_sensor_commands="$(arg fake_sensor_commands)" torque_constants="${[base_tc, shoulder_tc, elbow_tc, wrist1_tc, wrist2_tc, wrist3_tc]}" />
 </robot>

File: rbpodo_description/robots/rb5_850e_u.urdf (robot description, URDF)
Before this commit: robot rb20_1900es, 8 links, 7 joints
Links:
- link link0: geometry collision mesh filename=package://rbpodo_description/meshes/rb5_850e_u/collision/li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; visual mesh filename=package://rbpodo_description/meshes/rb5_850e_u/visual/link0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
- link link1: mass 15.48 -> 4.147; geometry collision mesh filename=package://rbpodo_description/meshes/rb5_850e_u/collision/li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; visual mesh filename=package://rbpodo_description/meshes/rb5_850e_u/visual/link1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
- link link2: mass 32.79 -> 9.633; geometry collision mesh filename=package://rbpodo_description/meshes/rb5_850e_u/collision/li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; visual mesh filename=package://rbpodo_description/meshes/rb5_850e_u/visual/link2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
- link link3: mass 8.371 -> 3.915; geometry collision mesh filename=package://rbpodo_description/meshes/rb5_850e_u/collision/li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; visual mesh filename=package://rbpodo_description/meshes/rb5_850e_u/visual/link3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
- link link4: mass 8.14 -> 1.452; geometry collision mesh filename=package://rbpodo_description/meshes/rb5_850e_u/collision/li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; visual mesh filename=package://rbpodo_description/meshes/rb5_850e_u/visual/link4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
- link link5: mass 1.924 -> 1.454; geometry collision mesh filename=package://rbpodo_description/meshes/rb5_850e_u/collision/li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; visual mesh filename=package://rbpodo_description/meshes/rb5_850e_u/visual/link5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
- link link6: mass 0.588 -> 0.243; geometry collision mesh filename=package://rbpodo_description/meshes/rb5_850e_u/collision/li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; visual mesh filename=package://rbpodo_description/meshes/rb5_850e_u/visual/link6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
Joints:
- joint base: origin xyz=0 0 0.241 rpy=0 0 0 -> xyz=0 0 0.1655 rpy=0 0 0
- joint elbow: origin xyz=0 0 0.885 rpy=0 0 0 -> xyz=0 0 0.425 rpy=0 0 0
- joint shoulder: origin xyz=0 -0.2545 0 rpy=0 0 0 -> xyz=0 0 0 rpy=0 0 0
- joint tcp_joint: origin xyz=0 0 0.13 rpy=0 0 0 -> xyz=0 -0.0967 0 rpy=0 0 0
- joint wrist1: axis 0 0 1 -> 0 1 0; origin xyz=0 0.1875 0 rpy=0 0 0 -> xyz=0 0 0.392 rpy=0 0 0
- joint wrist2: axis 0 1 0 -> 0 0 1; origin xyz=0 -0.1292 0.885 rpy=0 0 0 -> xyz=0 -0.1107 0.1107 rpy=0 0 0
- joint wrist3: axis 0 0 1 -> 0 1 0; origin xyz=0 0.1292 0 rpy=0 0 0 -> xyz=0 0 0 rpy=0 0 0

File: rbpodo_description/robots/rb5_850e_u.urdf.xacro (robot description, xacro)
@@ -1,4 +1,4 @@
 <?xml version='1.0' encoding='utf-8'?>
-<robot xmlns:xacro="http://www.ros.org/wiki/xacro" name="rb20_1900es">
+<robot xmlns:xacro="http://www.ros.org/wiki/xacro" name="rb5_850e_u">
   <xacro:include filename="$(find rbpodo_description)/robots/rb_6dof.xacro" />
   <xacro:include filename="$(find rbpodo_description)/robots/rb_6dof.ros2_control.xacro" />
@@ -6,5 +6,5 @@
   <xacro:arg name="robot_ip" default="10.0.2.7"/>
   <xacro:arg name="cb_simulation" default="true"/>
-  <xacro:arg name="use_fake_hardware" default="true"/>
+  <xacro:arg name="use_fake_hardware" default="false"/>
   <xacro:arg name="fake_sensor_commands" default="false"/>
   <!-- torque_constant = actual_torque_constant * gear_ratio -->
@@ -15,5 +15,5 @@
   <xacro:property name="wrist2_tc" value="${1}" />
   <xacro:property name="wrist3_tc" value="${1}" />
-  <xacro:rb_6dof model_id="rb20_1900es" prefix="$(arg prefix)" tcp_name="tcp" tcp_xyz="0 0 0.13" tcp_rpy="0 0 0" />
+  <xacro:rb_6dof model_id="rb5_850e_u" prefix="$(arg prefix)" tcp_name="tcp" tcp_xyz="0 -0.0967 0" tcp_rpy="0 0 0" />
   <xacro:rb_6dof_ros2_control prefix="$(arg prefix)" robot_ip="$(arg robot_ip)" cb_simulation="$(arg cb_simulation)" use_fake_hardware="$(arg use_fake_hardware)" fake_sensor_commands="$(arg fake_sensor_commands)" torque_constants="${[base_tc, shoulder_tc, elbow_tc, wrist1_tc, wrist2_tc, wrist3_tc]}" />
 </robot>
