Commit message: fix: rb20_1800e_u model added

File: rbpodo_description/robots/rb20_1800e_u.urdf.xacro (robot description, xacro)
@@ -1,4 +1,4 @@
 <?xml version='1.0' encoding='utf-8'?>
-<robot xmlns:xacro="http://www.ros.org/wiki/xacro" name="rb20_1900es">
+<robot xmlns:xacro="http://www.ros.org/wiki/xacro" name="rb20_1800e_u">
   <xacro:include filename="$(find rbpodo_description)/robots/rb_6dof.xacro" />
   <xacro:include filename="$(find rbpodo_description)/robots/rb_6dof.ros2_control.xacro" />
@@ -15,5 +15,5 @@
   <xacro:property name="wrist2_tc" value="${1}" />
   <xacro:property name="wrist3_tc" value="${1}" />
-  <xacro:rb_6dof model_id="rb20_1900es" prefix="$(arg prefix)" tcp_name="tcp" tcp_xyz="0 0 0.13" tcp_rpy="0 0 0" />
+  <xacro:rb_6dof model_id="rb20_1800e_u" prefix="$(arg prefix)" tcp_name="tcp" tcp_xyz="0 -0.13 0" tcp_rpy="0 0 0" />
   <xacro:rb_6dof_ros2_control prefix="$(arg prefix)" robot_ip="$(arg robot_ip)" cb_simulation="$(arg cb_simulation)" use_fake_hardware="$(arg use_fake_hardware)" fake_sensor_commands="$(arg fake_sensor_commands)" torque_constants="${[base_tc, shoulder_tc, elbow_tc, wrist1_tc, wrist2_tc, wrist3_tc]}" />
 </robot>

File: rbpodo_description/robots/rb20_1900es_u.urdf (robot description, URDF)
Before this commit: robot rb30_1400es, 8 links, 7 joints
Links:
- link link0: geometry collision mesh filename=package://rbpodo_description/meshes/rb20_1900es_u/collision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; visual mesh filename=package://rbpodo_description/meshes/rb20_1900es_u/visual/li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
- link link1: geometry collision mesh filename=package://rbpodo_description/meshes/rb20_1900es_u/collision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; visual mesh filename=package://rbpodo_description/meshes/rb20_1900es_u/visual/li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
- link link2: geometry collision mesh filename=package://rbpodo_description/meshes/rb20_1900es_u/collision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; visual mesh filename=package://rbpodo_description/meshes/rb20_1900es_u/visual/li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
- link link3: geometry collision mesh filename=package://rbpodo_description/meshes/rb20_1900es_u/collision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; visual mesh filename=package://rbpodo_description/meshes/rb20_1900es_u/visual/li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
- link link4: geometry collision mesh filename=package://rbpodo_description/meshes/rb20_1900es_u/collision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; visual mesh filename=package://rbpodo_description/meshes/rb20_1900es_u/visual/li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
- link link5: geometry collision mesh filename=package://rbpodo_description/meshes/rb20_1900es_u/collision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; visual mesh filename=package://rbpodo_description/meshes/rb20_1900es_u/visual/li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
- link link6: geometry collision mesh filename=package://rbpodo_description/meshes/rb20_1900es_u/collision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; visual mesh filename=package://rbpodo_description/meshes/rb20_1900es_u/visual/li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
Joints:
- joint elbow: origin xyz=0 0 0.630 rpy=0 0 0 -> xyz=0 0 0.885 rpy=0 0 0
- joint wrist2: origin xyz=0 -0.1292 0.640 rpy=0 0 0 -> xyz=0 -0.1292 0.885 rpy=0 0 0

File: rbpodo_description/robots/rb30_1400es_u.urdf (robot description, URDF)
Before this commit: robot rb20_1900es, 8 links, 7 joints
Links:
- link link0: geometry collision mesh filename=package://rbpodo_description/meshes/rb30_1400es_u/collision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; visual mesh filename=package://rbpodo_description/meshes/rb30_1400es_u/visual/li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
- link link1: geometry collision mesh filename=package://rbpodo_description/meshes/rb30_1400es_u/collision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; visual mesh filename=package://rbpodo_description/meshes/rb30_1400es_u/visual/li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
- link link2: geometry collision mesh filename=package://rbpodo_description/meshes/rb30_1400es_u/collision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; visual mesh filename=package://rbpodo_description/meshes/rb30_1400es_u/visual/li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
- link link3: geometry collision mesh filename=package://rbpodo_description/meshes/rb30_1400es_u/collision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; visual mesh filename=package://rbpodo_description/meshes/rb30_1400es_u/visual/li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
- link link4: geometry collision mesh filename=package://rbpodo_description/meshes/rb30_1400es_u/collision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; visual mesh filename=package://rbpodo_description/meshes/rb30_1400es_u/visual/li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
- link link5: geometry collision mesh filename=package://rbpodo_description/meshes/rb30_1400es_u/collision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; visual mesh filename=package://rbpodo_description/meshes/rb30_1400es_u/visual/li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
- link link6: geometry collision mesh filename=package://rbpodo_description/meshes/rb30_1400es_u/collision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; visual mesh filename=package://rbpodo_description/meshes/rb30_1400es_u/visual/li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
Joints:
- joint elbow: origin xyz=0 0 0.885 rpy=0 0 0 -> xyz=0 0 0.630 rpy=0 0 0
- joint wrist2: origin xyz=0 -0.1292 0.885 rpy=0 0 0 -> xyz=0 -0.1292 0.640 rpy=0 0 0

File: rbpodo_description/robots/rb30_1400es_u.urdf.xacro (robot description, xacro)
@@ -1,4 +1,4 @@
 <?xml version='1.0' encoding='utf-8'?>
-<robot xmlns:xacro="http://www.ros.org/wiki/xacro" name="rb30_1400es">
+<robot xmlns:xacro="http://www.ros.org/wiki/xacro" name="rb30_1400es_u">
   <xacro:include filename="$(find rbpodo_description)/robots/rb_6dof.xacro" />
   <xacro:include filename="$(find rbpodo_description)/robots/rb_6dof.ros2_control.xacro" />
@@ -15,5 +15,5 @@
   <xacro:property name="wrist2_tc" value="${1}" />
   <xacro:property name="wrist3_tc" value="${1}" />
-  <xacro:rb_6dof model_id="rb30_1400es" prefix="$(arg prefix)" tcp_name="tcp" tcp_xyz="0 0 0.13" tcp_rpy="0 0 0" />
+  <xacro:rb_6dof model_id="rb30_1400es_u" prefix="$(arg prefix)" tcp_name="tcp" tcp_xyz="0 0 0.13" tcp_rpy="0 0 0" />
   <xacro:rb_6dof_ros2_control prefix="$(arg prefix)" robot_ip="$(arg robot_ip)" cb_simulation="$(arg cb_simulation)" use_fake_hardware="$(arg use_fake_hardware)" fake_sensor_commands="$(arg fake_sensor_commands)" torque_constants="${[base_tc, shoulder_tc, elbow_tc, wrist1_tc, wrist2_tc, wrist3_tc]}" />
 </robot>
